File: WET_PCB_v2/currsense_DCDC.kicad_sch (KiCad schematic)
At the start: 8 parts, among them J1 Capacitor connector, U3 Opamp_Quad

Commit message: notees
Parts:
- removed D15, D16: 1N4004, Diode_THT:D_DO-15_P2.54mm_Vertical_CathodeUp, symbol Diode:1N4004
- added D25, D27: D_Zener, Diode_THT:D_DO-15_P2.54mm_Vertical_CathodeUp, symbol Device:D_Zener
Connections:
- net GND: now also D27.2 (A)
- net VDD_OPAMP: now also D25.1 (K)
- net currsense_ADC: now also D25.2 (A), D27.1 (K)
Other:
- note removed: "Shouldnt these be Zener diodes??"
Changed lines of the file:
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@@
 	(generator_version "10.0")
 	(paper "A4")
-	(text "Shouldnt these be Zener diodes??\n"
-		(exclude_from_sim no)
-		(at 136.144 63.246 0)
-		(effects
-			(font
-				(size 1.27 1.27)
-			)
-		)
-	)
 	(junction
 		(at 93.98 58.42)
@@
 	)
 	(junction
-		(at 69.85 55.88)
-		(diameter 0)
-		(color 0 0 0 0)
-	)
-	(junction
 		(at 104.14 58.42)
 		(diameter 0)
@@
 		(color 0 0 0 0)
 	)
+	(junction
+		(at 68.58 55.88)
+		(diameter 0)
+		(color 0 0 0 0)
+	)
 	(wire
 		(pts
@@
 	(wire
 		(pts
-			(xy 73.66 40.64) (xy 69.85 40.64)
-		)
-		(stroke
-			(width 0)
-			(type default)
-		)
-	)
-	(wire
-		(pts
-			(xy 69.85 40.64) (xy 69.85 55.88)
+			(xy 73.66 40.64) (xy 68.58 40.64)
+		)
+		(stroke
+			(width 0)
+			(type default)
+		)
+	)
+	(wire
+		(pts
+			(xy 68.58 40.64) (xy 68.58 55.88)
 		)
 		(stroke
@@
 	(wire
 		(pts
-			(xy 69.85 55.88) (xy 72.39 55.88)
-		)
-		(stroke
-			(width 0)
-			(type default)
-		)
-	)
-	(wire
-		(pts
-			(xy 63.5 55.88) (xy 69.85 55.88)
+			(xy 63.5 55.88) (xy 68.58 55.88)
 		)
 		(stroke
@@
 		(pts
 			(xy 104.14 45.72) (xy 104.14 49.53)
+		)
+		(stroke
+			(width 0)
+			(type default)
+		)
+	)
+	(wire
+		(pts
+			(xy 68.58 55.88) (xy 72.39 55.88)
 		)
 		(stroke
@@
 	)
 	(symbol
+		(lib_id "Device:D_Zener")
+		(at 104.14 53.34 270)
+		(unit 1)
+		(body_style 1)
+		(exclude_from_sim no)
+		(in_bom yes)
+		(on_board yes)
+		(in_pos_files yes)
+		(dnp no)
+		(fields_autoplaced yes)
+		(property "Reference" "D25"
+			(at 106.68 52.0699 90)
+			(show_name no)
+			(do_not_autoplace no)
+			(effects
+				(font
+					(size 1.27 1.27)
+				)
+				(justify left)
+			)
+		)
+		(property "Value" "D_Zener"
+			(at 106.68 54.6099 90)
+			(show_name no)
+			(do_not_autoplace no)
+			(effects
+				(font
+					(size 1.27 1.27)
+				)
+				(justify left)
+			)
+		)
+		(property "Footprint" "Diode_THT:D_DO-15_P2.54mm_Vertical_CathodeUp"
+			(at 104.14 53.34 0)
+			(hide yes)
+			(show_name no)
+			(do_not_autoplace no)
+			(effects
+				(font
+					(size 1.27 1.27)
+				)
+			)
+		)
+		(property "Datasheet" ""
+			(at 104.14 53.34 0)
+			(hide yes)
+			(show_name no)
+			(do_not_autoplace no)
+			(effects
+				(font
+					(size 1.27 1.27)
+				)
+			)
+		)
+		(property "Description" "Zener diode"
+			(at 104.14 53.34 0)
+			(hide yes)
+			(show_name no)
+			(do_not_autoplace no)
+			(effects
+				(font
+					(size 1.27 1.27)
+				)
+			)
+		)
+		(pin "2"
+		)
+		(pin "1"
+		)
+		(instances
+			(project "WET_PCB_v2"
+				(path "/13451c35-1666-47d9-9525-8d8125ba1cf3/12f67741-eb23-4832-9e03-479bbedcb04e"
+					(reference "D25")
+					(unit 1)
+				)
+				(path "/13451c35-1666-47d9-9525-8d8125ba1cf3/6ecc05b2-84d4-404f-84e6-8cc19742ad68"
+					(reference "D26")
+					(unit 1)
+				)
+			)
+		)
+	)
+	(symbol
 		(lib_id "Device:R")
 		(at 77.47 40.64 90)
@@
 	)
 	(symbol
-		(lib_id "Diode:1N4004")
-		(at 104.14 53.34 90)
-		(mirror x)
-		(unit 1)
-		(body_style 1)
-		(exclude_from_sim no)
-		(in_bom yes)
-		(on_board yes)
-		(in_pos_files yes)
-		(dnp no)
-		(fields_autoplaced yes)
-		(property "Reference" "D15"
-			(at 106.68 52.0699 90)
-			(show_name no)
-			(do_not_autoplace no)
-			(effects
-				(font
-					(size 1.27 1.27)
-				)
-				(justify right)
-			)
-		)
-		(property "Value" "1N4004"
-			(at 106.68 54.6099 90)
-			(show_name no)
-			(do_not_autoplace no)
-			(effects
-				(font
-					(size 1.27 1.27)
-				)
-				(justify right)
-			)
-		)
-		(property "Footprint" "Diode_THT:D_DO-15_P2.54mm_Vertical_CathodeUp"
-			(at 108.585 53.34 0)
-			(hide yes)
-			(show_name no)
-			(do_not_autoplace no)
-			(effects
-				(font
-					(size 1.27 1.27)
-				)
-			)
-		)
-		(property "Datasheet" "http://www.vishay.com/docs/88503/1n4001.pdf"
-			(at 104.14 53.34 0)
-			(hide yes)
-			(show_name no)
-			(do_not_autoplace no)
-			(effects
-				(font
-					(size 1.27 1.27)
-				)
-			)
-		)
-		(property "Description" "400V 1A General Purpose Rectifier Diode, DO-41"
-			(at 104.14 53.34 0)
-			(hide yes)
-			(show_name no)
-			(do_not_autoplace no)
-			(effects
-				(font
-					(size 1.27 1.27)
-				)
-			)
-		)
-		(property "Sim.Device" "D"
-			(at 104.14 53.34 0)
-			(hide yes)
-			(show_name no)
-			(do_not_autoplace no)
-			(effects
-				(font
-					(size 1.27 1.27)
-				)
-			)
-		)
-		(property "Sim.Pins" "1=K 2=A"
-			(at 104.14 53.34 0)
-			(hide yes)
-			(show_name no)
-			(do_not_autoplace no)
-			(effects
-				(font
-					(size 1.27 1.27)
-				)
-			)
-		)
-		(pin "1"
-		)
-		(pin "2"
-		)
-		(instances
-			(project "WET_PCB_v2"
-				(path "/13451c35-1666-47d9-9525-8d8125ba1cf3/12f67741-eb23-4832-9e03-479bbedcb04e"
-					(reference "D15")
-					(unit 1)
-				)
-				(path "/13451c35-1666-47d9-9525-8d8125ba1cf3/6ecc05b2-84d4-404f-84e6-8cc19742ad68"
-					(reference "D17")
-					(unit 1)
-				)
-			)
-		)
-	)
-	(symbol
 		(lib_id "power:GND")
 		(at 104.14 71.12 0)
@@
 	)
 	(symbol
-		(lib_id "Diode:1N4004")
-		(at 104.14 64.77 90)
-		(mirror x)
+		(lib_id "Device:D_Zener")
+		(at 104.14 64.77 270)
 		(unit 1)
 		(body_style 1)
@@
 		(in_pos_files yes)
 		(dnp no)
-		(property "Reference" "D16"
+		(fields_autoplaced yes)
+		(property "Reference" "D27"
 			(at 106.68 63.4999 90)
 			(show_name no)
@@
 					(size 1.27 1.27)
 				)
-				(justify right)
-			)
-		)
-		(property "Value" "1N4004"
+				(justify left)
+			)
+		)
+		(property "Value" "D_Zener"
 			(at 106.68 66.0399 90)
 			(show_name no)
@@
 					(size 1.27 1.27)
 				)
-				(justify right)
+				(justify left)
 			)
 		)
 		(property "Footprint" "Diode_THT:D_DO-15_P2.54mm_Vertical_CathodeUp"
-			(at 108.585 64.77 0)
-			(hide yes)
-			(show_name no)
-			(do_not_autoplace no)
-			(effects
-				(font
-					(size 1.27 1.27)
-				)
-			)
-		)
-		(property "Datasheet" "http://www.vishay.com/docs/88503/1n4001.pdf"
 			(at 104.14 64.77 0)
 			(hide yes)
@@
 			)
 		)
-		(property "Description" "400V 1A General Purpose Rectifier Diode, DO-41"
+		(property "Datasheet" ""
 			(at 104.14 64.77 0)
 			(hide yes)
@@
 			)
 		)
-		(property "Sim.Device" "D"
+		(property "Description" "Zener diode"
 			(at 104.14 64.77 0)
 			(hide yes)
@@
 			)
 		)
-		(property "Sim.Pins" "1=K 2=A"
-			(at 104.14 64.77 0)
-			(hide yes)
-			(show_name no)
-			(do_not_autoplace no)
-			(effects
-				(font
-					(size 1.27 1.27)
-				)
-			)
+		(pin "2"
 		)
 		(pin "1"
-		)
-		(pin "2"
 		)
 		(instances
 			(project "WET_PCB_v2"
 				(path "/13451c35-1666-47d9-9525-8d8125ba1cf3/12f67741-eb23-4832-9e03-479bbedcb04e"
-					(reference "D16")
+					(reference "D27")
 					(unit 1)
 				)
 				(path "/13451c35-1666-47d9-9525-8d8125ba1cf3/6ecc05b2-84d4-404f-84e6-8cc19742ad68"
-					(reference "D18")
-					(unit 1)
-				)
+					(reference "D28")
+					(unit 1)
+				)

Commit message: redid part of layout inverter
Parts:
- R21, R22, R23, R24: footprint Resistor_THT:R_Axial_DIN0207_L6.3mm_D2.5mm_P7.62mm_Horizontal -> Resistor_SMD:R_0805_2012Metric_Pad1.20x1.40mm_HandSolder
Other:
- moved on the sheet: R22
Changed lines of the file:
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@@
 	(wire
 		(pts
-			(xy 73.66 40.64) (xy 68.58 40.64)
-		)
-		(stroke
-			(width 0)
-			(type default)
-		)
-	)
-	(wire
-		(pts
-			(xy 68.58 40.64) (xy 68.58 55.88)
+			(xy 73.66 48.26) (xy 68.58 48.26)
+		)
+		(stroke
+			(width 0)
+			(type default)
+		)
+	)
+	(wire
+		(pts
+			(xy 68.58 48.26) (xy 68.58 55.88)
 		)
 		(stroke
@@
 	(wire
 		(pts
-			(xy 90.17 40.64) (xy 90.17 58.42)
-		)
-		(stroke
-			(width 0)
-			(type default)
-		)
-	)
-	(wire
-		(pts
-			(xy 81.28 40.64) (xy 90.17 40.64)
+			(xy 90.17 48.26) (xy 90.17 58.42)
+		)
+		(stroke
+			(width 0)
+			(type default)
+		)
+	)
+	(wire
+		(pts
+			(xy 81.28 48.26) (xy 90.17 48.26)
 		)
 		(stroke
@@
 			)
 		)
-		(property "Footprint" "Resistor_THT:R_Axial_DIN0207_L6.3mm_D2.5mm_P7.62mm_Horizontal"
+		(property "Footprint" "Resistor_SMD:R_0805_2012Metric_Pad1.20x1.40mm_HandSolder"
 			(at 59.69 62.738 90)
 			(hide yes)
@@
 	(symbol
 		(lib_id "Device:R")
-		(at 77.47 40.64 90)
+		(at 77.47 48.26 90)
 		(unit 1)
 		(body_style 1)
@@
 		(fields_autoplaced yes)
 		(property "Reference" "R22"
-			(at 77.47 34.29 90)
+			(at 77.47 41.91 90)
 			(show_name no)
 			(do_not_autoplace no)
@@
 		)
 		(property "Value" "R"
-			(at 77.47 36.83 90)
-			(show_name no)
-			(do_not_autoplace no)
-			(effects
-				(font
-					(size 1.27 1.27)
-				)
-			)
-		)
-		(property "Footprint" "Resistor_THT:R_Axial_DIN0207_L6.3mm_D2.5mm_P7.62mm_Horizontal"
-			(at 77.47 42.418 90)
+			(at 77.47 44.45 90)
+			(show_name no)
+			(do_not_autoplace no)
+			(effects
+				(font
+					(size 1.27 1.27)
+				)
+			)
+		)
+		(property "Footprint" "Resistor_SMD:R_0805_2012Metric_Pad1.20x1.40mm_HandSolder"
+			(at 77.47 50.038 90)
 			(hide yes)
 			(show_name no)
@@
 		)
 		(property "Datasheet" ""
-			(at 77.47 40.64 0)
+			(at 77.47 48.26 0)
 			(hide yes)
 			(show_name no)
@@
 		)
 		(property "Description" "Resistor"
-			(at 77.47 40.64 0)
+			(at 77.47 48.26 0)
 			(hide yes)
 			(show_name no)
@@
 			)
 		)
-		(property "Footprint" "Resistor_THT:R_Axial_DIN0207_L6.3mm_D2.5mm_P7.62mm_Horizontal"
+		(property "Footprint" "Resistor_SMD:R_0805_2012Metric_Pad1.20x1.40mm_HandSolder"
 			(at 70.358 64.77 90)
 			(hide yes)
@@
 		(dnp no)
 		(property "Reference" "U3"
-			(at 78.74 59.6901 0)
+			(at 81.026 54.356 0)
 			(show_name no)
 			(do_not_autoplace no)
@@
 		(property "Value" "Opamp_Quad"
 			(at 77.724 51.562 0)
+			(hide yes)
 			(show_name no)
 			(do_not_autoplace no)
@@
 			)
 		)
-		(property "Footprint" "Resistor_THT:R_Axial_DIN0207_L6.3mm_D2.5mm_P7.62mm_Horizontal"
+		(property "Footprint" "Resistor_SMD:R_0805_2012Metric_Pad1.20x1.40mm_HandSolder"
 			(at 59.69 57.658 90)
 			(hide yes)

Commit message: didnt watch the lecture but made progress ig
Parts:
- J1: footprint (none) -> Connector_PinSocket_2.54mm:PinSocket_1x02_P2.54mm_Vertical
Changed lines of the file:
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@@
 			)
 		)
-		(property "Footprint" ""
+		(property "Footprint" "Connector_PinSocket_2.54mm:PinSocket_1x02_P2.54mm_Vertical"
 			(at 93.98 66.04 0)
 			(hide yes)
