File: WET_PCB_v2/12v5V.kicad_sch (KiCad schematic)
At the start: 0 parts

Commit message: before i prob fuck up everything bc clearance
Parts:
- added C10: C0.1uF, Capacitor_THT:C_Disc_D4.3mm_W1.9mm_P5.00mm, symbol Device:C
- added C9: C0.33uF, Capacitor_THT:C_Disc_D4.3mm_W1.9mm_P5.00mm, symbol Device:C
- added U6: L7805, Package_TO_SOT_THT:TO-220-3_Vertical, symbol Regulator_Linear:L7805
Connections:
- net Vin_12V: now also C9.1, U6.1 (IN)
- net Vout_5V: now also C10.1, U6.3 (OUT)
- new net GND: C10.2, C9.2, U6.2 (GND)
