File: WET_PCB_v2/decoration.kicad_sch (KiCad schematic)
At the start: 24 parts, among them J19 Fuse holder or smth to hold t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, J20 Fuse holder or smth to hold t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, J21 Fuse holder or smth to hold t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, J22 Fuse holder or smth to hold t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, J23 Fuse holder or smth to hold t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, J24 Fuse holder or smth to hold t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, J25 Fuse holder or smth to hold t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, J26 Fuse holder or smth to hold t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, J27 Fuse holder or smth to hold t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, J28 Fuse holder or smth to hold t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, J29 Fuse holder or smth to hold t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, J30 Fuse holder or smth to hold t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

Commit message: finished and added some drawings
Parts:
- removed J25, J26: Fuse holder or smth to hold tube, TestPoint:TestPoint_Loop_D2.60mm_Drill0.9mm_Beaded, symbol Connector:Conn_01x02_Socket
- renumbered J19 to MNT1, J28 to MNT10, J29 to MNT11, J30 to MNT12, J20 to MNT2, J21 to MNT3, J22 to MNT4, J23 to MNT5, J24 to MNT6, J27 to MNT9
Connections:
- no-connect marks 24 -> 20
Changed lines of the file:
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@@
-	)
-	(no_connect
-		(at 151.13 74.93)
 	)
 	(no_connect
@@
 	)
 	(no_connect
-		(at 151.13 85.09)
-	)
-	(no_connect
-		(at 151.13 82.55)
-	)
-	(no_connect
 		(at 134.62 86.36)
 	)
 	(no_connect
 		(at 151.13 106.68)
-	)
-	(no_connect
-		(at 151.13 72.39)
 	)
 	(no_connect
@@
 		(dnp no)
 		(fields_autoplaced yes)
-		(property "Reference" "J23"
+		(property "Reference" "MNT5"
 			(at 140.97 129.5399 0)
 			(show_name no)
@@
 			(project "WET_PCB_v2"
 				(path "/13451c35-1666-47d9-9525-8d8125ba1cf3/79e5e86e-dc26-4d0b-a087-2027a5880c08"
-					(reference "J23")
+					(reference "MNT5")
 					(unit 1)
 				)
@@
 		(dnp no)
 		(fields_autoplaced yes)
-		(property "Reference" "J19"
+		(property "Reference" "MNT1"
 			(at 140.97 76.1999 0)
 			(show_name no)
@@
 			(project "WET_PCB_v2"
 				(path "/13451c35-1666-47d9-9525-8d8125ba1cf3/79e5e86e-dc26-4d0b-a087-2027a5880c08"
-					(reference "J19")
+					(reference "MNT1")
 					(unit 1)
 				)
@@
 		(dnp no)
 		(fields_autoplaced yes)
-		(property "Reference" "J21"
+		(property "Reference" "MNT3"
 			(at 140.97 96.5199 0)
 			(show_name no)
@@
 			(project "WET_PCB_v2"
 				(path "/13451c35-1666-47d9-9525-8d8125ba1cf3/79e5e86e-dc26-4d0b-a087-2027a5880c08"
-					(reference "J21")
+					(reference "MNT3")
 					(unit 1)
 				)
@@
 	(symbol
 		(lib_id "Connector:Conn_01x02_Socket")
-		(at 156.21 82.55 0)
-		(unit 1)
-		(body_style 1)
-		(exclude_from_sim no)
-		(in_bom yes)
-		(on_board yes)
-		(in_pos_files yes)
-		(dnp no)
-		(fields_autoplaced yes)
-		(property "Reference" "J26"
-			(at 157.48 82.5499 0)
-			(show_name no)
-			(do_not_autoplace no)
-			(effects
-				(font
-					(size 1.27 1.27)
-				)
-				(justify left)
-			)
-		)
-		(property "Value" "Fuse holder or smth to hold tube"
-			(at 157.48 85.0899 0)
-			(hide yes)
-			(show_name no)
-			(do_not_autoplace no)
-			(effects
-				(font
-					(size 1.27 1.27)
-				)
-				(justify left)
-			)
-		)
-		(property "Footprint" "TestPoint:TestPoint_Loop_D2.60mm_Drill0.9mm_Beaded"
-			(at 156.21 82.55 0)
-			(hide yes)
-			(show_name no)
-			(do_not_autoplace no)
-			(effects
-				(font
-					(size 1.27 1.27)
-				)
-			)
-		)
-		(property "Datasheet" ""
-			(at 156.21 82.55 0)
-			(hide yes)
-			(show_name no)
-			(do_not_autoplace no)
-			(effects
-				(font
-					(size 1.27 1.27)
-				)
-			)
-		)
-		(property "Description" "Generic connector, single row, 01x02, script generated"
-			(at 156.21 82.55 0)
-			(hide yes)
-			(show_name no)
-			(do_not_autoplace no)
-			(effects
-				(font
-					(size 1.27 1.27)
-				)
-			)
-		)
-		(pin "2"
-		)
-		(pin "1"
-		)
-		(instances
-			(project "WET_PCB_v2"
-				(path "/13451c35-1666-47d9-9525-8d8125ba1cf3/79e5e86e-dc26-4d0b-a087-2027a5880c08"
-					(reference "J26")
-					(unit 1)
-				)
-			)
-		)
-	)
-	(symbol
-		(lib_id "Connector:Conn_01x02_Socket")
 		(at 157.48 118.11 0)
 		(unit 1)
@@
 		(dnp no)
 		(fields_autoplaced yes)
-		(property "Reference" "J30"
+		(property "Reference" "MNT12"
 			(at 158.75 118.1099 0)
 			(show_name no)
@@
 			(project "WET_PCB_v2"
 				(path "/13451c35-1666-47d9-9525-8d8125ba1cf3/79e5e86e-dc26-4d0b-a087-2027a5880c08"
-					(reference "J30")
-					(unit 1)
-				)
-			)
-		)
-	)
-	(symbol
-		(lib_id "Connector:Conn_01x02_Socket")
-		(at 156.21 72.39 0)
-		(unit 1)
-		(body_style 1)
-		(exclude_from_sim no)
-		(in_bom yes)
-		(on_board yes)
-		(in_pos_files yes)
-		(dnp no)
-		(fields_autoplaced yes)
-		(property "Reference" "J25"
-			(at 157.48 72.3899 0)
-			(show_name no)
-			(do_not_autoplace no)
-			(effects
-				(font
-					(size 1.27 1.27)
-				)
-				(justify left)
-			)
-		)
-		(property "Value" "Fuse holder or smth to hold tube"
-			(at 157.48 74.9299 0)
-			(hide yes)
-			(show_name no)
-			(do_not_autoplace no)
-			(effects
-				(font
-					(size 1.27 1.27)
-				)
-				(justify left)
-			)
-		)
-		(property "Footprint" "TestPoint:TestPoint_Loop_D2.60mm_Drill0.9mm_Beaded"
-			(at 156.21 72.39 0)
-			(hide yes)
-			(show_name no)
-			(do_not_autoplace no)
-			(effects
-				(font
-					(size 1.27 1.27)
-				)
-			)
-		)
-		(property "Datasheet" ""
-			(at 156.21 72.39 0)
-			(hide yes)
-			(show_name no)
-			(do_not_autoplace no)
-			(effects
-				(font
-					(size 1.27 1.27)
-				)
-			)
-		)
-		(property "Description" "Generic connector, single row, 01x02, script generated"
-			(at 156.21 72.39 0)
-			(hide yes)
-			(show_name no)
-			(do_not_autoplace no)
-			(effects
-				(font
-					(size 1.27 1.27)
-				)
-			)
-		)
-		(pin "2"
-		)
-		(pin "1"
-		)
-		(instances
-			(project "WET_PCB_v2"
-				(path "/13451c35-1666-47d9-9525-8d8125ba1cf3/79e5e86e-dc26-4d0b-a087-2027a5880c08"
-					(reference "J25")
+					(reference "MNT12")
 					(unit 1)
 				)
@@
 		(dnp no)
 		(fields_autoplaced yes)
-		(property "Reference" "J22"
+		(property "Reference" "MNT4"
 			(at 140.97 107.9499 0)
 			(show_name no)
@@
 			(project "WET_PCB_v2"
 				(path "/13451c35-1666-47d9-9525-8d8125ba1cf3/79e5e86e-dc26-4d0b-a087-2027a5880c08"
-					(reference "J22")
+					(reference "MNT4")
 					(unit 1)
 				)
@@
 		(dnp no)
 		(fields_autoplaced yes)
-		(property "Reference" "J20"
+		(property "Reference" "MNT2"
 			(at 140.97 86.3599 0)
 			(show_name no)
@@
 			(project "WET_PCB_v2"
 				(path "/13451c35-1666-47d9-9525-8d8125ba1cf3/79e5e86e-dc26-4d0b-a087-2027a5880c08"
-					(reference "J20")
+					(reference "MNT2")
 					(unit 1)
 				)
@@
 		(dnp no)
 		(fields_autoplaced yes)
-		(property "Reference" "J29"
+		(property "Reference" "MNT11"
 			(at 157.48 125.7299 0)
 			(show_name no)
@@
 			(project "WET_PCB_v2"
 				(path "/13451c35-1666-47d9-9525-8d8125ba1cf3/79e5e86e-dc26-4d0b-a087-2027a5880c08"
-					(reference "J29")
+					(reference "MNT11")
 					(unit 1)
 				)
@@
 		(dnp no)
 		(fields_autoplaced yes)
-		(property "Reference" "J24"
+		(property "Reference" "MNT6"
 			(at 142.24 121.9199 0)
 			(show_name no)
@@
 			(project "WET_PCB_v2"
 				(path "/13451c35-1666-47d9-9525-8d8125ba1cf3/79e5e86e-dc26-4d0b-a087-2027a5880c08"
-					(reference "J24")
+					(reference "MNT6")
 					(unit 1)
 				)
@@
 		(dnp no)
 		(fields_autoplaced yes)
-		(property "Reference" "J28"
+		(property "Reference" "MNT10"
 			(at 157.48 104.1399 0)
 			(show_name no)
@@
 			(project "WET_PCB_v2"
 				(path "/13451c35-1666-47d9-9525-8d8125ba1cf3/79e5e86e-dc26-4d0b-a087-2027a5880c08"
-					(reference "J28")
+					(reference "MNT10")
 					(unit 1)
 				)
@@
 		(dnp no)
 		(fields_autoplaced yes)
-		(property "Reference" "J27"
+		(property "Reference" "MNT9"
 			(at 157.48 92.7099 0)
 			(show_name no)
@@
 			(project "WET_PCB_v2"
 				(path "/13451c35-1666-47d9-9525-8d8125ba1cf3/79e5e86e-dc26-4d0b-a087-2027a5880c08"
-					(reference "J27")
-					(unit 1)
-				)
+					(reference "MNT9")
+					(unit 1)
+				)
