File: WET_PCB_v2/GateDriver.kicad_sch (KiCad schematic)
At the start: 11 parts, among them U4 IR2110

Commit message: notees
Other:
- note added: "add second cap"
Changed lines of the file:
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@@
+		)
+	)
+	(text "add second cap"
+		(exclude_from_sim no)
+		(at 71.628 52.832 0)
+		(effects
+			(font
+				(size 1.27 1.27)
+			)
 		)
 	)

Commit message: redid part of layout inverter
Other:
- note added: "check cap orientation"
- note removed: "add second cap"
- note removed: "does this have to be this hugeass diode?"
Changed lines of the file:
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@@
 	(generator_version "10.0")
 	(paper "A4")
-	(text "does this have to be this hugeass diode?\n"
+	(text "check cap orientation\n"
 		(exclude_from_sim no)
-		(at 102.362 40.132 0)
+		(at 130.048 68.834 0)
 		(effects
 			(font
-				(size 1.27 1.27)
-			)
-		)
-	)
-	(text "add second cap"
-		(exclude_from_sim no)
-		(at 71.628 52.832 0)
-		(effects
-			(font

Commit message: before i prob fuck up everything bc clearance
Parts:
- added C24: C322C104K5R5TA, Capacitor_THT:C_Disc_D4.3mm_W1.9mm_P5.00mm, symbol C322C104K5R5TA:C322C104K5R5TA
Connections:
- net GND: now also C24.1
- net VDD_Driver_DCDC: now also C24.2

Commit message: veel routes weinig goeds
Connections:
- net DCDC_Driver_SD renamed SD
Changed lines of the file:
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@@
 		)
 	)
-	(hierarchical_label "DCDC_Driver_SD"
+	(hierarchical_label "SD"
 		(shape input)
 		(at 62.23 72.39 180)
