File: WET_PCB_v2/WET_PCB_v2.kicad_sch (KiCad schematic)
At the start: 24 parts, among them J10 Conn_01x09_Pin, J11 Conn_01x09_Pin, J2 Conn_01x09_Pin, J3 Conn_01x09_Pin, J4 XT60, J5 Barrel jack, J6 Pluggable Terminal Block, J7 Pluggable Terminal Block, J8 Jumper, U3 Opamp_Quad

Commit message: notees
Parts:
- J4: value XT60 -> Pluggable terminal block; footprint Connector_AMASS:AMASS_XT60PW-F_1x02_P7.20mm_Horizontal -> Connector_Phoenix_GMSTB:PhoenixContact_GMSTBA_2,5_2-G-7,62_1x02_P7.62mm_Horizontal
Other:
- added sheet curr_sense_coil (curr_sense_coil.kicad_sch)
- note added: "add 0ohm"
- note added: "add footprint to add wires trough current measurement"
- note added: "add resitor footprint"
- note added: "look for other UV LEDs"

Commit message: redid part of layout inverter
Parts:
- added R37, R38, R39, R40: R0, Resistor_SMD:R_0805_2012Metric_Pad1.20x1.40mm_HandSolder, symbol Device:R
- R5, R6: footprint Resistor_THT:R_Axial_DIN0204_L3.6mm_D1.6mm_P1.90mm_Vertical -> Resistor_SMD:R_0805_2012Metric_Pad1.20x1.40mm_HandSolder
- R7, R8: footprint Resistor_THT:R_Axial_DIN0207_L6.3mm_D2.5mm_P15.24mm_Horizontal -> Resistor_SMD:R_2512_6332Metric_Pad1.40x3.35mm_HandSolder
Connections:
- net GND: now also R38.2, R39.2, R40.2
- net VPP: now also R37.1
- new net DCDC/DCDC_Driver_SD: R38.1
- new net currsense_DCDC/Shunt_from_source: R37.2
- new net inverter/Inv_Driver_Left_SD: R39.1
- new net inverter/Inv_Driver_Right_SD: R40.1

Commit message: didnt watch the lecture but made progress ig
Parts:
- added J16: POGO1, Connector_PinHeader_1.00mm:PinHeader_1x01_P1.00mm_Vertical, symbol Connector:Conn_01x01_Pin
- added J21: POGO2, Connector_PinHeader_1.00mm:PinHeader_1x01_P1.00mm_Vertical, symbol Connector:Conn_01x01_Pin
- added R43: R0, Resistor_SMD:R_0805_2012Metric_Pad1.20x1.40mm_HandSolder, symbol Device:R
- J4: value Pluggable terminal block -> Power input
- J6: value Pluggable Terminal Block -> Coil plug
Connections:
- net VPP: no longer R37.1, R7.1
- net currsense_DCDC/Shunt_to_load: now also R43.2
- net DCDC/Vin_DCDC+ renamed DCDC/currsense_FET_side
- net DCDC/currsense_FET_side: now also R43.1
- new net: J16.1 (Pin_1), U7.19 (POGO_PRG)
- new net: J21.1 (Pin_1), U7.20 (POGO_PRG)
- new net DCDC/currsense_cap_side: R37.1, R7.1
Other:
- sheet DCDC ports: added currsense_FET_side, currsense_cap_side; removed none

Commit message: i think it fits holy
Parts:
- added R44, R45: R0, Resistor_SMD:R_0805_2012Metric_Pad1.20x1.40mm_HandSolder, symbol Device:R
Connections:
- net DCDC/DCDC_coil_circuit_side: now also J6.2 (Pin_2); no longer J6.1 (Pin_1)
- net DCDC/DCDC_coil_input_side: now also J6.1 (Pin_1); no longer J6.2 (Pin_2)
- net DCDC/VoutDCDC: now also R8.2, R45.1
- net currsense_inv/Shunt_from_source: now also R44.2; no longer R8.1
- net currsense_inv/Shunt_to_load: now also R45.2; no longer R8.2
- new net inverter/Vin_Inverter: R44.1, R8.1
Other:
- moved on the sheet: J10, J11, J16, J2, J21, J3, J6, J7, R37, R38, R39, R40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

Commit message: lecture done
Changed lines of the file:
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@@
 	(wire
 		(pts
+			(xy 172.72 110.49) (xy 176.53 110.49)
+		)
+		(stroke
+			(width 0)
+			(type default)
+		)
+	)
+	(wire
+		(pts
 			(xy 246.38 115.57) (xy 243.84 115.57)
 		)
@@
 	(wire
 		(pts
-			(xy 172.72 99.06) (xy 172.72 110.49)
-		)
-		(stroke
-			(width 0)
-			(type default)
-		)
-	)
-	(wire
-		(pts
 			(xy 49.53 57.15) (xy 62.23 57.15)
 		)
@@
 		)
 	)
+	(label "ADC1_IN5"
+		(at 176.53 110.49 0)
+		(effects
+			(font
+				(size 1.27 1.27)
+			)
+			(justify left bottom)
+		)
+	)
 	(label "TIM3_CH1"
 		(at 213.36 88.9 270)
@@
 		)
 	)
+	(label "ADC1_IN4"
+		(at 168.91 27.94 180)
+		(effects
+			(font
+				(size 1.27 1.27)
+			)
+			(justify right bottom)
+		)
+	)
 	(label "TIM3_CH2"
 		(at 224.79 88.9 270)
@@
 	)
 	(label "ADC1_IN5"
-		(at 175.26 128.27 0)
-		(effects
-			(font
-				(size 1.27 1.27)
-			)
-			(justify left bottom)
-		)
-	)
-	(label "ADC1_IN5"
 		(at 306.07 142.24 180)
 		(effects
@@
 		)
 	)
-	(label "ADC1_IN4"
+	(label "ADC1_IN0"
+		(at 175.26 128.27 0)
+		(effects
+			(font
+				(size 1.27 1.27)
+			)
+			(justify left bottom)
+		)
+	)
+	(label "ADC1_IN1"
 		(at 246.38 115.57 0)
 		(effects
@@
 		)
 	)
-	(label "ADC1_IN1"
-		(at 168.91 27.94 180)
-		(effects
-			(font
-				(size 1.27 1.27)
-			)
-			(justify right bottom)
-		)
-	)
 	(label "TIM1_CH4"
 		(at 31.75 106.68 0)
@@
 	)
 	(group ""
-		(members "a17383a4-d27f-4c25-9e0c-b0df1856b8d8" "b0cb1397-fac0-444b-95f5-30e95b8f9aaf"
-			"e547f70c-7bec-4117-9e0a-e594b69335eb"
-		)
+		(members "a17383a4-d27f-4c25-9e0c-b0df1856b8d8" "e547f70c-7bec-4117-9e0a-e594b69335eb")
 	)
 	(sheet

Commit message: before i prob fuck up everything bc clearance
Parts:
- removed C17, C20, C21: C_Polarized, Capacitor_THT:CP_Radial_D5.0mm_P2.00mm, symbol Device:C_Polarized
- added J26: Vsense_ADC1_IN1, Connector_PinHeader_1.00mm:PinHeader_1x01_P1.00mm_Vertical, symbol Connector:Conn_01x01_Pin
- added R48, R49, R50, R51, R52, R53, R54, R55, R56, R57: R0, Resistor_SMD:R_0805_2012Metric_Pad1.20x1.40mm_HandSolder, symbol Device:R
Connections:
- net ADC1_IN0: now also R55.2
- net ADC1_IN1: now also R57.2
- net ADC1_IN5: now also R54.2
- net TIM14_CH1: now also R49.2
- net TIM1_CH4: now also R48.2
- net TIM3_CH1: now also R50.2, R53.2
- net TIM3_CH2: now also R51.2, R52.2
- net inverter/Vout_Inverter_+: now also J7.1 (Pin_1); no longer J7.2 (Pin_2)
- net inverter/Vout_Inverter_-: now also J7.2 (Pin_2); no longer J7.1 (Pin_1)
- net voltsense_inverter/Vsense_in: now also J26.1 (Pin_1)
- net GPIO_A12 renamed ADC1_IN16
- net ADC1_IN16: now also R56.2
- new net DCDC/DCDC_Driver_Hin: R48.1
- new net DCDC/DCDC_Driver_Lin: R49.1
- new net curr_sense_coil/transducer_out: R56.1
- new net currsense_DCDC/currsense_ADC: R54.1
- new net inverter/Inv_Driver_Left_Hin: R50.1
- new net inverter/Inv_Driver_Left_Lin: R51.1
- new net inverter/Inv_Driver_Right_Hin: R52.1
- new net inverter/Inv_Driver_Right_Lin: R53.1
- new net voltsense_DCDC/Vsense_ADC: R55.1
- new net voltsense_inverter/Vsense_ADC: R57.1
- no-connect marks 1 -> 0
Other:
- sheet curr_sense_coil ports: added VDD_clippingdiode, transducer_out, transducer_power; removed none
- note removed: "the caps have random footprints so they appear in the layout designer"
- moved on the sheet: J7

Commit message: im gonna start to route and probably revert to this version at least 5 times
Connections:
- net inverter/Vout_Inverter_+: now also J7.2 (Pin_2); no longer J7.1 (Pin_1)
- net inverter/Vout_Inverter_-: now also J7.1 (Pin_1); no longer J7.2 (Pin_2)
Other:
- sheet decoration ports: added UVLED5, UVLED6; removed none
Changed lines of the file:
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@@
 	)
 	(junction
+		(at 29.21 114.3)
+		(diameter 0)
+		(color 0 0 0 0)
+	)
+	(junction
 		(at 294.64 142.24)
 		(diameter 0)
@@
 	)
 	(junction
+		(at 29.21 116.84)
+		(diameter 0)
+		(color 0 0 0 0)
+	)
+	(junction
 		(at 29.21 106.68)
 		(diameter 0)
@@
 	(wire
 		(pts
+			(xy 26.67 116.84) (xy 29.21 116.84)
+		)
+		(stroke
+			(width 0)
+			(type default)
+		)
+	)
+	(wire
+		(pts
 			(xy 132.08 162.56) (xy 132.08 161.29)
 		)
@@
 	(wire
 		(pts
+			(xy 26.67 119.38) (xy 29.21 119.38)
+		)
+		(stroke
+			(width 0)
+			(type default)
+		)
+	)
+	(wire
+		(pts
 			(xy 373.38 149.86) (xy 387.35 149.86)
 		)
@@
 	(wire
 		(pts
+			(xy 29.21 119.38) (xy 29.21 116.84)
+		)
+		(stroke
+			(width 0)
+			(type default)
+		)
+	)
+	(wire
+		(pts
 			(xy 29.21 109.22) (xy 29.21 111.76)
 		)
@@
 	(wire
 		(pts
+			(xy 29.21 116.84) (xy 29.21 114.3)
+		)
+		(stroke
+			(width 0)
+			(type default)
+		)
+	)
+	(wire
+		(pts
 			(xy 86.36 78.74) (xy 86.36 77.47)
 		)
@@
 	)
 	(symbol
-		(lib_id "Connector:Conn_01x02_Pin")
-		(at 251.46 57.15 0)
-		(mirror y)
-		(unit 1)
-		(body_style 1)
-		(exclude_from_sim no)
-		(in_bom yes)
-		(on_board yes)
-		(in_pos_files yes)
-		(dnp no)
-		(property "Reference" "J7"
-			(at 249.936 60.452 0)
-			(show_name no)
-			(do_not_autoplace no)
-			(effects
-				(font
-					(size 1.27 1.27)
-				)
-			)
-		)
-		(property "Value" "Pluggable Terminal Block"
-			(at 249.174 63.754 0)
-			(show_name no)
-			(do_not_autoplace no)
-			(effects
-				(font
-					(size 1.27 1.27)
-				)
-			)
-		)
-		(property "Footprint" "Connector_Phoenix_GMSTB:PhoenixContact_GMSTBA_2,5_2-G-7,62_1x02_P7.62mm_Horizontal"
-			(at 251.46 57.15 0)
-			(hide yes)
-			(show_name no)
-			(do_not_autoplace no)
-			(effects
-				(font
-					(size 1.27 1.27)
-				)
-			)
-		)
-		(property "Datasheet" ""
-			(at 251.46 57.15 0)
-			(hide yes)
-			(show_name no)
-			(do_not_autoplace no)
-			(effects
-				(font
-					(size 1.27 1.27)
-				)
-			)
-		)
-		(property "Description" "Generic connector, single row, 01x02, script generated"
-			(at 251.46 57.15 0)
-			(hide yes)
-			(show_name no)
-			(do_not_autoplace no)
-			(effects
-				(font
-					(size 1.27 1.27)
-				)
-			)
-		)
-		(pin "1"
-		)
-		(pin "2"
-		)
-		(instances
-			(project "WET_PCB_v2"
-				(path "/13451c35-1666-47d9-9525-8d8125ba1cf3"
-					(reference "J7")
-					(unit 1)
-				)
-			)
-		)
-	)
-	(symbol
 		(lib_id "C322C104K5R5TA:C322C104K5R5TA")
 		(at 86.36 78.74 270)
@@
 	)
 	(symbol
+		(lib_id "Connector:Conn_01x02_Pin")
+		(at 251.46 59.69 180)
+		(unit 1)
+		(body_style 1)
+		(exclude_from_sim no)
+		(in_bom yes)
+		(on_board yes)
+		(in_pos_files yes)
+		(dnp no)
+		(property "Reference" "J7"
+			(at 249.936 56.388 0)
+			(show_name no)
+			(do_not_autoplace no)
+			(effects
+				(font
+					(size 1.27 1.27)
+				)
+			)
+		)
+		(property "Value" "Pluggable Terminal Block"
+			(at 249.174 53.086 0)
+			(show_name no)
+			(do_not_autoplace no)
+			(effects
+				(font
+					(size 1.27 1.27)
+				)
+			)
+		)
+		(property "Footprint" "Connector_Phoenix_GMSTB:PhoenixContact_GMSTBA_2,5_2-G-7,62_1x02_P7.62mm_Horizontal"
+			(at 251.46 59.69 0)
+			(hide yes)
+			(show_name no)
+			(do_not_autoplace no)
+			(effects
+				(font
+					(size 1.27 1.27)
+				)
+			)
+		)
+		(property "Datasheet" ""
+			(at 251.46 59.69 0)
+			(hide yes)
+			(show_name no)
+			(do_not_autoplace no)
+			(effects
+				(font
+					(size 1.27 1.27)
+				)
+			)
+		)
+		(property "Description" "Generic connector, single row, 01x02, script generated"
+			(at 251.46 59.69 0)
+			(hide yes)
+			(show_name no)
+			(do_not_autoplace no)
+			(effects
+				(font
+					(size 1.27 1.27)
+				)
+			)
+		)
+		(pin "1"
+		)
+		(pin "2"
+		)
+		(instances
+			(project "WET_PCB_v2"
+				(path "/13451c35-1666-47d9-9525-8d8125ba1cf3"
+					(reference "J7")
+					(unit 1)
+				)
+			)
+		)
+	)
+	(symbol
 		(lib_id "Device:R")
 		(at 190.5 58.42 270)
@@
 	(sheet
 		(at 13.97 104.14)
-		(size 12.7 12.7)
+		(size 12.7 17.78)
 		(exclude_from_sim no)
 		(in_bom yes)
@@
 		)
 		(property "Sheetfile" "decoration.kicad_sch"
-			(at 13.97 117.4246 0)
+			(at 13.97 122.5046 0)
 			(hide yes)
 			(show_name no)
@@
 			(effects
 				(font
+					(size 1.27 1.27)
+				)
+				(justify right)
+			)
+		)
+		(pin "UVLED5" input
+			(at 26.67 116.84 0)
+			(effects
+				(font
+					(size 1.27 1.27)
+				)
+				(justify right)
+			)
+		)
+		(pin "UVLED6" input
+			(at 26.67 119.38 0)
+			(effects
+				(font

Commit message: veel routes weinig goeds
Connections:
- net DCDC/currsense_FET_side: now also R7.1; no longer R7.2
- net DCDC/currsense_cap_side: now also R7.2; no longer R7.1
- net curr_sense_coil/transducer_out renamed curr_sense_coil/transducer_out_scaled
Other:
- sheet curr_sense_coil ports: added transducer_out_scaled; removed transducer_out
- moved on the sheet: R38, R7
Changed lines of the file:
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@@
 	)
 	(junction
+		(at 149.86 85.09)
+		(diameter 0)
+		(color 0 0 0 0)
+	)
+	(junction
 		(at 194.31 58.42)
 		(diameter 0)
@@
 		(color 0 0 0 0)
 	)
-	(junction
-		(at 149.86 85.09)
-		(diameter 0)
-		(color 0 0 0 0)
-	)
 	(wire
 		(pts
@@
 	(wire
 		(pts
+			(xy 134.62 144.78) (xy 134.62 146.05)
+		)
+		(stroke
+			(width 0)
+			(type default)
+		)
+	)
+	(wire
+		(pts
 			(xy 53.34 77.47) (xy 69.85 77.47)
 		)
@@
 	(wire
 		(pts
+			(xy 175.26 81.28) (xy 175.26 80.01)
+		)
+		(stroke
+			(width 0)
+			(type default)
+		)
+	)
+	(wire
+		(pts
 			(xy 29.21 114.3) (xy 26.67 114.3)
 		)
@@
 	(wire
 		(pts
+			(xy 134.62 149.86) (xy 134.62 151.13)
+		)
+		(stroke
+			(width 0)
+			(type default)
+		)
+	)
+	(wire
+		(pts
 			(xy 373.38 152.4) (xy 387.35 152.4)
 		)
@@
 	(wire
 		(pts
+			(xy 175.26 90.17) (xy 175.26 88.9)
+		)
+		(stroke
+			(width 0)
+			(type default)
+		)
+	)
+	(wire
+		(pts
 			(xy 69.85 77.47) (xy 86.36 77.47)
 		)
@@
 	(symbol
 		(lib_id "Device:R")
-		(at 153.67 85.09 90)
+		(at 153.67 85.09 270)
 		(unit 1)
 		(body_style 1)
@@
 		)
 		(property "Footprint" "Resistor_SMD:R_2512_6332Metric_Pad1.40x3.35mm_HandSolder"
-			(at 153.67 86.868 90)
+			(at 153.67 83.312 90)
 			(hide yes)
 			(show_name no)
@@
 		)
 		(property "Value" "Vsense_ADC1_IN1"
-			(at 196.342 132.08 0)
+			(at 189.738 133.604 0)
 			(show_name no)
 			(do_not_autoplace no)
@@
 	(symbol
 		(lib_id "Device:R")
-		(at 175.26 83.82 0)
+		(at 175.26 85.09 0)
 		(unit 1)
 		(body_style 1)
@@
 		(fields_autoplaced yes)
 		(property "Reference" "R38"
-			(at 177.8 82.5499 0)
+			(at 177.8 83.8199 0)
 			(show_name no)
 			(do_not_autoplace no)
@@
 		)
 		(property "Value" "R0"
-			(at 177.8 85.0899 0)
+			(at 177.8 86.3599 0)
 			(show_name no)
 			(do_not_autoplace no)
@@
 		)
 		(property "Footprint" "Resistor_SMD:R_0805_2012Metric_Pad1.20x1.40mm_HandSolder"
-			(at 173.482 83.82 90)
+			(at 173.482 85.09 90)
 			(hide yes)
 			(show_name no)
@@
 		)
 		(property "Datasheet" ""
-			(at 175.26 83.82 0)
+			(at 175.26 85.09 0)
 			(hide yes)
 			(show_name no)
@@
 		)
 		(property "Description" "Resistor"
-			(at 175.26 83.82 0)
+			(at 175.26 85.09 0)
 			(hide yes)
 			(show_name no)
@@
 	(symbol
 		(lib_id "power:GND")
-		(at 175.26 87.63 0)
+		(at 175.26 90.17 0)
 		(unit 1)
 		(body_style 1)
@@
 		(fields_autoplaced yes)
 		(property "Reference" "#PWR051"
-			(at 175.26 93.98 0)
+			(at 175.26 96.52 0)
 			(hide yes)
 			(show_name no)
@@
 		)
 		(property "Value" "GND"
-			(at 175.26 92.71 0)
+			(at 175.26 95.25 0)
 			(show_name no)
 			(do_not_autoplace no)
@@
 		)
 		(property "Footprint" ""
-			(at 175.26 87.63 0)
+			(at 175.26 90.17 0)
 			(hide yes)
 			(show_name no)
@@
 		)
 		(property "Datasheet" ""
-			(at 175.26 87.63 0)
+			(at 175.26 90.17 0)
 			(hide yes)
 			(show_name no)
@@
 		)
 		(property "Description" "Power symbol creates a global label with name \"GND\" , ground"
-			(at 175.26 87.63 0)
+			(at 175.26 90.17 0)
 			(hide yes)
 			(show_name no)
@@
 		(in_pos_files yes)
 		(dnp no)
-		(fields_autoplaced yes)
 		(property "Reference" "R49"
-			(at 175.26 82.5499 0)
+			(at 175.26 83.8199 0)
 			(show_name no)
 			(do_not_autoplace no)
@@
 		)
 		(property "Value" "R0"
-			(at 175.26 85.0899 0)
+			(at 175.26 86.3599 0)
 			(show_name no)
 			(do_not_autoplace no)
@@
 		(in_pos_files yes)
 		(dnp no)
-		(fields_autoplaced yes)
 		(property "Reference" "R48"
-			(at 172.72 82.5499 0)
+			(at 172.72 83.8199 0)
 			(show_name no)
 			(do_not_autoplace no)
@@
 			)
 		)
-		(pin "transducer_out" output
+		(pin "transducer_out_scaled" output
 			(at 172.72 167.64 0)
 			(effects
