File: WET_PCB_v2/WET_PCB_v2.kicad_pcb (KiCad board)
At the start: 2 copper layers, 100 x 80 mm, 102 parts, among them J10 Conn_01x09_Pin, J11 Conn_01x09_Pin, J17 Capacitor connector, J18 Capacitor connector, J19 Capacitor connector, J2 Conn_01x09_Pin, J20 Capacitor connector, J3 Conn_01x09_Pin, J4 XT60, J5 Barrel jack, J6 Pluggable Terminal Block, J7 Pluggable Terminal Block, J8 Jumper, Q1 IRF530NPBF, Q2 IRF530NPBF, Q3 IRF530NPBF, Q4 IRF530NPBF, Q5 Q_NMOS_GDS, Q6 Q_NMOS_GDS, U1 IR2110, U2 IR2110, U3 Opamp_Quad, U4 IR2110

Commit message: redid part of layout inverter
Parts:
- added C22: C_Polarized, Capacitor_THT:C_Radial_D12.5mm_H20.0mm_P5.00mm, F.Cu at (89.0, 73.0)
- added C8: B32529C1104K000, Capacitor_THT:C_Rect_L7.0mm_W2.5mm_P5.00mm, F.Cu at (104.3, 96.4)
- added D25: D_Zener, Diode_THT:D_DO-15_P2.54mm_Vertical_CathodeUp, F.Cu at (102.4, 68.6)
- added D26: D_Zener, Diode_THT:D_DO-15_P2.54mm_Vertical_CathodeUp, F.Cu at (95.4, 84.6)
- added D27: D_Zener, Diode_THT:D_DO-15_P2.54mm_Vertical_CathodeUp, F.Cu at (102.4, 73.7)
- added D28: D_Zener, Diode_THT:D_DO-15_P2.54mm_Vertical_CathodeUp, F.Cu at (95.4, 89.8)
- added D29: D_Zener, Diode_THT:D_DO-15_P2.54mm_Vertical_CathodeUp, F.Cu at (104.4, 84.6)
- added D30: D_Zener, Diode_THT:D_DO-15_P2.54mm_Vertical_CathodeUp, F.Cu at (104.4, 89.8)
- added D31: D_Zener, Diode_THT:D_DO-15_P2.54mm_Vertical_CathodeUp, F.Cu at (86.4, 84.6)
- added D32: D_Zener, Diode_THT:D_DO-15_P2.54mm_Vertical_CathodeUp, F.Cu at (86.4, 89.8)
- added HS1: Heatsink, Heatsink:Heatsink_AAVID_Extruded_531002B02100G_34.9x12.7mm_H25.4mm, F.Cu at (258.0, 53.5)
- added HS2: Heatsink, Heatsink:Heatsink_AAVID_Extruded_531002B02100G_34.9x12.7mm_H25.4mm, F.Cu at (208.3, 48.8)
- added HS3: Heatsink, Heatsink:Heatsink_AAVID_Extruded_531002B02100G_34.9x12.7mm_H25.4mm, F.Cu at (299.0, 123.2)
- added HS4: Heatsink, Heatsink:Heatsink_AAVID_Extruded_531002B02100G_34.9x12.7mm_H25.4mm, F.Cu at (315.8, 123.2)
- added HS5: Heatsink, Heatsink:Heatsink_AAVID_Extruded_531002B02100G_34.9x12.7mm_H25.4mm, F.Cu at (315.8, 86.7)
- added HS6: Heatsink, Heatsink:Heatsink_AAVID_Extruded_531002B02100G_34.9x12.7mm_H25.4mm, F.Cu at (299.0, 86.7)
- added R37: R0, Resistor_SMD:R_0805_2012Metric_Pad1.20x1.40mm_HandSolder, F.Cu at (111.9, 67.5)
- added R38: R0, Resistor_SMD:R_0805_2012Metric_Pad1.20x1.40mm_HandSolder, F.Cu at (111.9, 70.4)
- added R39: R0, Resistor_SMD:R_0805_2012Metric_Pad1.20x1.40mm_HandSolder, F.Cu at (111.9, 73.4)
- added R40: R0, Resistor_SMD:R_0805_2012Metric_Pad1.20x1.40mm_HandSolder, F.Cu at (111.9, 76.3)
- D19, D20, D21, D22: footprint LED_SMD:LED_1W_3W_R8 -> LED_SMD:LED_PLCC-2_3.4x3.0mm_AK
- J4: value XT60 -> Pluggable terminal block; footprint Connector_AMASS:AMASS_XT60PW-F_1x02_P7.20mm_Horizontal -> Connector_Phoenix_GMSTB:PhoenixContact_GMSTBA_2,5_2-G-7,62_1x02_P7.62mm_Horizontal
- R1, R2, R21, R22, R23, R24, R25, R26, R27, R28, R29, R3, R30, R31, R32, R33, R34, R35, R36, R4: footprint Resistor_THT:R_Axial_DIN0207_L6.3mm_D2.5mm_P7.62mm_Horizontal -> Resistor_SMD:R_0805_2012Metric_Pad1.20x1.40mm_HandSolder
- R5, R6: footprint Resistor_THT:R_Axial_DIN0204_L3.6mm_D1.6mm_P1.90mm_Vertical -> Resistor_SMD:R_0805_2012Metric_Pad1.20x1.40mm_HandSolder
- R7, R8: footprint Resistor_THT:R_Axial_DIN0207_L6.3mm_D2.5mm_P15.24mm_Horizontal -> Resistor_SMD:R_2512_6332Metric_Pad1.40x3.35mm_HandSolder
- moved C5 131.7 mm to (338.4, 106.6), turned to -90 degrees
- moved U2 128.5 mm to (333.2, 97.8), turned to 0 degrees
- moved C6 126.7 mm to (335.6, 106.6), turned to -90 degrees
- moved D4 117.3 mm to (328.9, 104.1)
- moved D5 114.3 mm to (333.3, 87.8), turned to 90 degrees
- moved R13 111.8 mm to (330.3, 89.2), turned to 180 degrees
- moved C7 111.3 mm to (328.5, 111.6)
- moved Q3 108.8 mm to (320.1, 89.2), turned to 90 degrees
- moved R15 103.0 mm to (322.7, 84.2), turned to 0 degrees
- moved D6 82.1 mm to (333.1, 124.7), turned to 90 degrees
- moved R14 81.3 mm to (330.3, 125.8), turned to 180 degrees
- moved R16 78.3 mm to (322.8, 120.6), turned to 0 degrees
- moved Q4 74.8 mm to (320.1, 125.7), turned to 90 degrees
- moved C3 61.2 mm to (304.8, 152.1)
- moved C8 61.2 mm to (295.3, 152.1)
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Connections:
- C1 pad 2: /inverter/VDD_Inverter -> +5V
- C14 pad 1: /DCDC/DCDC_coil_circuit_side -> /DCDC/Gatedriver/Vs_node
- C15 pad 1: /DCDC/DCDC_coil_circuit_side -> /DCDC/Gatedriver/Vs_node
- C5 pad 2: /inverter/VDD_Inverter -> +5V
- Q5 pad 2: /DCDC/DCDC_coil_circuit_side -> /DCDC/Gatedriver/Vs_node
- Q6 pad 2: /DCDC/DCDC_coil_circuit_side -> /DCDC/VoutDCDC
- Q6 pad 3: /DCDC/VoutDCDC -> /DCDC/Gatedriver/Vs_node
- R19 pad 1: /DCDC/DCDC_coil_circuit_side -> /DCDC/Gatedriver/Vs_node
- R21 pad 1: /DCDC/DCDC_coil_input_side -> /currsense_DCDC/Shunt_to_load
- R23 pad 1: VPP -> /currsense_DCDC/Shunt_from_source
- U1 pad 11: GND -> /inverter/Inv_Driver_Left_SD
- U1 pad 9: /inverter/VDD_Inverter -> +5V
- U2 pad 11: GND -> /inverter/Inv_Driver_Right_SD
- U2 pad 9: /inverter/VDD_Inverter -> +5V
- U4 pad 5: /DCDC/DCDC_coil_circuit_side -> /DCDC/Gatedriver/Vs_node

Commit message: didnt watch the lecture but made progress ig
Parts:
- removed the C8 at (295.3, 152.1)
- removed D15, D16, D17, D18, D23, D24, D7, D8: 1N4004, Diode_THT:D_DO-15_P2.54mm_Vertical_CathodeUp
- added C23: C_Polarized, Capacitor_THT:C_Radial_D12.5mm_H20.0mm_P5.00mm, F.Cu at (130.7, 41.8)
- added J1: Capacitor connector, Connector_PinSocket_2.54mm:PinSocket_1x02_P2.54mm_Vertical, F.Cu at (128.4, 53.1)
- added J16: POGO1, Connector_PinHeader_1.00mm:PinHeader_1x01_P1.00mm_Vertical, F.Cu at (232.6, 150.6)
- added J21: POGO2, Connector_PinHeader_1.00mm:PinHeader_1x01_P1.00mm_Vertical, F.Cu at (230.0, 148.8)
- added J9: Capacitor connector, Connector_PinSocket_2.54mm:PinSocket_1x02_P2.54mm_Vertical, F.Cu at (135.0, 53.1)
- added R41: R0, Resistor_SMD:R_0805_2012Metric_Pad1.20x1.40mm_HandSolder, F.Cu at (165.4, 50.9)
- added R42: R0, Resistor_SMD:R_0805_2012Metric_Pad1.20x1.40mm_HandSolder, F.Cu at (165.4, 55.8)
- added R43: R0, Resistor_SMD:R_0805_2012Metric_Pad1.20x1.40mm_HandSolder, F.Cu at (165.4, 45.9)
- C4, C7, D1, D4, D9: moved to B.Cu
- J4: value Pluggable terminal block -> Power input
- J6: value Pluggable Terminal Block -> Coil plug
- moved D5 174.7 mm to (168.4, 145.6)
- moved R15 164.8 mm to (171.6, 150.1), turned to 90 degrees
- moved R13 162.7 mm to (176.6, 142.5), turned to -90 degrees
- moved U2 158.7 mm to (182.8, 148.5), turned to 90 degrees
- moved HS5 158.2 mm to (174.1, 157.0), turned to 180 degrees
- moved Q3 156.9 mm to (176.6, 152.7), turned to 180 degrees
- moved C12 154.8 mm to (85.7, 107.6)
- moved C5 151.3 mm to (191.6, 143.3), turned to 0 degrees
- moved C6 149.3 mm to (191.6, 146.1), turned to 0 degrees
- moved D4 146.8 mm to (190.1, 151.8), turned to 180 degrees
- moved C7 139.3 mm to (195.0, 151.4), turned to 0 degrees
- moved C11 138.2 mm to (65.8, 109.7)
- moved D6 130.0 mm to (204.8, 145.5)
- moved Q1 129.7 mm to (170.9, 122.7), turned to 0 degrees
- moved HS6 129.5 mm to (173.4, 118.4), turned to 0 degrees
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Connections:
- C14 pad 1: /DCDC/Gatedriver/Vs_node -> /DCDC/currsense_FET_side
- C15 pad 1: /DCDC/Gatedriver/Vs_node -> /DCDC/currsense_FET_side
- D25 pad 2: /ADC1_IN1 -> /currsense_DCDC/currsense_ADC
- D27 pad 1: /ADC1_IN1 -> /currsense_DCDC/currsense_ADC
- J6 pad 2: /DCDC/DCDC_coil_input_side -> VPP
- Q5 pad 2: /DCDC/Gatedriver/Vs_node -> /DCDC/currsense_FET_side
- Q6 pad 3: /DCDC/Gatedriver/Vs_node -> /DCDC/currsense_FET_side
- R19 pad 1: /DCDC/Gatedriver/Vs_node -> /DCDC/currsense_FET_side
- R22 pad 2: /ADC1_IN1 -> /currsense_DCDC/currsense_ADC
- R36 pad 1: Net-(U3A--) -> Net-(R36-Pad1)
- R37 pad 1: VPP -> /DCDC/DCDC_coil_circuit_side
- R4 pad 1: Net-(U3B-in2-) -> Net-(U3B-out2)
- R7 pad 1: VPP -> /DCDC/DCDC_coil_circuit_side
- R7 pad 2: /DCDC/DCDC_coil_input_side -> /DCDC/currsense_FET_side
- U3 pad 1: Net-(U3A--) -> Net-(R36-Pad1)
- U3 pad 7: Net-(U3B-in2-) -> Net-(U3B-out2)
- U3 pad 8: /ADC1_IN1 -> /currsense_DCDC/currsense_ADC
- U4 pad 5: /DCDC/Gatedriver/Vs_node -> /DCDC/currsense_FET_side

Commit message: i think it fits holy
Parts:
- added R44: R0, Resistor_SMD:R_0805_2012Metric_Pad1.20x1.40mm_HandSolder, B.Cu at (182.0, 115.0)
- added R45: R0, Resistor_SMD:R_0805_2012Metric_Pad1.20x1.40mm_HandSolder, B.Cu at (181.8, 110.0)
- C11, C12, C15, C22, C23, J9, R25, R26, R27, R28, R8: moved to B.Cu
- moved D28 178.5 mm to (243.0, 147.0), turned to 180 degrees
- moved D26 176.1 mm to (240.4, 142.0)
- moved C11 169.2 mm to (234.0, 91.0), turned to 0 degrees
- moved C22 162.2 mm to (228.0, 99.0), turned to 180 degrees
- moved J7 160.0 mm to (160.8, 101.2), turned to -90 degrees
- moved C3 146.7 mm to (165.0, 107.5), turned to 90 degrees
- moved J9 143.5 mm to (240.0, 151.0), turned to -90 degrees
- moved J4 142.1 mm to (255.0, 90.7)
- moved J5 139.0 mm to (249.7, 110.9), turned to 90 degrees
- moved D12 128.3 mm to (246.0, 90.1)
- moved R33 121.7 mm to (246.0, 94.0)
- moved C18 120.6 mm to (209.0, 106.0)
- moved C20 120.6 mm to (203.0, 106.0)
- moved U3 120.6 mm to (213.6, 103.2)
- moved R28 116.7 mm to (212.0, 114.0), turned to 0 degrees
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Connections:
- J6 pad 1: /DCDC/DCDC_coil_circuit_side -> VPP
- J6 pad 2: VPP -> /DCDC/DCDC_coil_circuit_side
- Q1 pad 2: /DCDC/VoutDCDC -> /inverter/Vin_Inverter
- Q3 pad 2: /DCDC/VoutDCDC -> /inverter/Vin_Inverter
- R8 pad 1: /currsense_inv/Shunt_from_source -> /inverter/Vin_Inverter
- R8 pad 2: /currsense_inv/Shunt_to_load -> /DCDC/VoutDCDC

Commit message: lecture done
Parts:
- R21, R22, R23, R24, R35, R37, R4, R43, R7: moved to B.Cu
- moved J18 188.0 mm to (252.0, 148.0)
- moved D31 181.8 mm to (245.5, 109.0)
- moved D32 181.7 mm to (245.5, 113.2)
- moved D27 176.6 mm to (241.0, 148.0), turned to 180 degrees
- moved D29 174.5 mm to (245.4, 148.0)
- moved D25 174.4 mm to (238.4, 143.0)
- moved D30 173.6 mm to (247.9, 143.8), turned to 180 degrees
- moved J1 128.5 mm to (246.0, 105.0), turned to 90 degrees
- moved R36 121.8 mm to (246.4, 151.0)
- moved R24 107.6 mm to (216.0, 103.0), turned to 90 degrees
- moved R23 103.8 mm to (215.0, 100.0), turned to 0 degrees
- moved R22 100.6 mm to (218.0, 107.0)
- moved R34 99.0 mm to (243.0, 95.0), turned to 180 degrees
- moved R21 97.9 mm to (218.0, 103.0)
- moved R35 97.6 mm to (222.0, 107.0), turned to 90 degrees
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Connections:
- D25 pad 2: /currsense_DCDC/currsense_ADC -> /ADC1_IN5
- D26 pad 2: /ADC1_IN1 -> /ADC1_IN4
- D27 pad 1: /currsense_DCDC/currsense_ADC -> /ADC1_IN5
- D28 pad 1: /ADC1_IN1 -> /ADC1_IN4
- D29 pad 1: /ADC1_IN5 -> /ADC1_IN0
- D30 pad 2: /ADC1_IN5 -> /ADC1_IN0
- D31 pad 2: /ADC1_IN4 -> /ADC1_IN1
- D32 pad 1: /ADC1_IN4 -> /ADC1_IN1
- J1 pad 2: /currsense_DCDC/currsense_ADC -> /ADC1_IN5
- J17 pad 2: /ADC1_IN4 -> /ADC1_IN1
- J18 pad 2: /ADC1_IN5 -> /ADC1_IN0
- J9 pad 2: /ADC1_IN1 -> /ADC1_IN4
- R22 pad 2: /currsense_DCDC/currsense_ADC -> /ADC1_IN5
- R28 pad 2: /ADC1_IN1 -> /ADC1_IN4
- R36 pad 2: /ADC1_IN5 -> /ADC1_IN0
- R4 pad 2: /ADC1_IN4 -> /ADC1_IN1
- U3 pad 14: /ADC1_IN1 -> /ADC1_IN4
- U3 pad 8: /currsense_DCDC/currsense_ADC -> /ADC1_IN5

Commit message: before i prob fuck up everything bc clearance
Parts:
- removed C17, C20, C21: C_Polarized, Capacitor_THT:CP_Radial_D5.0mm_P2.00mm
- removed C3: B32529C1104K000, Capacitor_THT:C_Rect_L7.0mm_W2.5mm_P5.00mm
- added C10: C0.1uF, Capacitor_THT:C_Disc_D4.3mm_W1.9mm_P5.00mm, F.Cu at (251.5, 127.5)
- added C24: C322C104K5R5TA, Capacitor_THT:C_Disc_D4.3mm_W1.9mm_P5.00mm, F.Cu at (177.5, 94.5)
- added C25: C322C104K5R5TA, Capacitor_THT:C_Disc_D4.3mm_W1.9mm_P5.00mm, F.Cu at (256.5, 136.5)
- added C26: C322C104K5R5TA, Capacitor_THT:C_Disc_D4.3mm_W1.9mm_P5.00mm, F.Cu at (181.0, 135.5)
- added C9: C0.33uF, Capacitor_THT:C_Disc_D4.3mm_W1.9mm_P5.00mm, B.Cu at (251.5, 125.0)
- added D33: D_Zener, Diode_THT:D_DO-15_P2.54mm_Vertical_CathodeUp, F.Cu at (243.5, 132.0)
- added D34: D_Zener, Diode_THT:D_DO-15_P2.54mm_Vertical_CathodeUp, F.Cu at (243.6, 136.5)
- added J22: LA55_GND, Connector_PinSocket_2.54mm:PinSocket_1x01_P2.54mm_Horizontal, B.Cu at (248.0, 142.9)
- added J23: LA55_M, Connector_PinSocket_2.54mm:PinSocket_1x01_P2.54mm_Horizontal, B.Cu at (248.0, 148.0)
- added J24: LA55_+, Connector_PinSocket_2.54mm:PinSocket_1x01_P2.54mm_Horizontal, B.Cu at (248.0, 120.0)
- added J25: Capacitor connector, Connector_PinSocket_2.54mm:PinSocket_1x02_P2.54mm_Vertical, F.Cu at (242.0, 147.2)
- added J26: Vsense_ADC1_IN1, Connector_PinHeader_1.00mm:PinHeader_1x01_P1.00mm_Vertical, F.Cu at (194.2, 112.0)
- added R46: R, Resistor_SMD:R_0805_2012Metric_Pad1.20x1.40mm_HandSolder, F.Cu at (250.5, 151.0)
- added R47: R, Resistor_SMD:R_0805_2012Metric_Pad1.20x1.40mm_HandSolder, F.Cu at (254.5, 151.0)
- added R48: R0, Resistor_SMD:R_0805_2012Metric_Pad1.20x1.40mm_HandSolder, B.Cu at (237.0, 106.5)
- added R49: R0, Resistor_SMD:R_0805_2012Metric_Pad1.20x1.40mm_HandSolder, B.Cu at (239.0, 106.5)
- added R50: R0, Resistor_SMD:R_0805_2012Metric_Pad1.20x1.40mm_HandSolder, B.Cu at (232.0, 106.5)
- added R51: R0, Resistor_SMD:R_0805_2012Metric_Pad1.20x1.40mm_HandSolder, B.Cu at (241.0, 106.5)
- added R52: R0, Resistor_SMD:R_0805_2012Metric_Pad1.20x1.40mm_HandSolder, B.Cu at (243.0, 106.5)
- added R53: R0, Resistor_SMD:R_0805_2012Metric_Pad1.20x1.40mm_HandSolder, B.Cu at (234.0, 106.5)
- added R54: R0, Resistor_SMD:R_0805_2012Metric_Pad1.20x1.40mm_HandSolder, F.Cu at (242.0, 106.5)
- added R55: R0, Resistor_SMD:R_0805_2012Metric_Pad1.20x1.40mm_HandSolder, F.Cu at (235.0, 144.5)
- added R56: R0, Resistor_SMD:R_0805_2012Metric_Pad1.20x1.40mm_HandSolder, F.Cu at (240.0, 106.5)
- added R57: R0, Resistor_SMD:R_0805_2012Metric_Pad1.20x1.40mm_HandSolder, F.Cu at (235.0, 142.0)
- added U5: LA55-P, Sensor_Current:LEM_LA25-P, F.Cu at (268.5, 147.9)
- added U6: L7805, Package_TO_SOT_THT:TO-220-3_Vertical, B.Cu at (250.7, 116.6)
- C1, C18, C19, C2, C5, C6, R1, R2, R3, R38, R39, R40: moved to B.Cu
- moved C19 175.0 mm to (206.0, 107.0), turned to 180 degrees
- moved J8 140.1 mm to (255.5, 130.5), turned to -90 degrees
- moved C16 137.9 mm to (248.0, 125.0), turned to 180 degrees
- moved R40 120.5 mm to (189.5, 144.0), turned to -90 degrees
- moved R39 119.8 mm to (193.0, 134.5), turned to 90 degrees
- moved J17 117.3 mm to (230.3, 144.5), turned to -90 degrees
- moved J19 115.9 mm to (230.3, 140.5), turned to -90 degrees
- moved R38 102.9 mm to (189.5, 98.5)
- moved R3 102.8 mm to (198.5, 107.0), turned to 90 degrees
- moved R2 100.9 mm to (201.5, 113.5), turned to 0 degrees
- moved R1 96.5 mm to (197.5, 113.5), turned to 0 degrees
- moved C8 92.2 mm to (165.5, 136.5), turned to -90 degrees
- moved R42 65.2 mm to (212.5, 101.0)
- moved R41 60.0 mm to (200.0, 101.0), turned to 180 degrees
- moved J7 34.0 mm to (160.8, 135.2)
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Connections:
- net /GPIO_A12 renamed /ADC1_IN16
- D25 pad 2: /ADC1_IN5 -> /currsense_DCDC/currsense_ADC
- D27 pad 1: /ADC1_IN5 -> /currsense_DCDC/currsense_ADC
- D29 pad 1: /ADC1_IN0 -> /voltsense_DCDC/Vsense_ADC
- D30 pad 1: +5V -> /voltsense_DCDC/VDD_OPAMP
- D30 pad 2: /ADC1_IN0 -> /voltsense_DCDC/Vsense_ADC
- D31 pad 2: /ADC1_IN1 -> /voltsense_inverter/Vsense_ADC
- D32 pad 1: /ADC1_IN1 -> /voltsense_inverter/Vsense_ADC
- J1 pad 2: /ADC1_IN5 -> /currsense_DCDC/currsense_ADC
- J17 pad 2: /ADC1_IN1 -> /voltsense_inverter/Vsense_ADC
- J18 pad 2: /ADC1_IN0 -> /voltsense_DCDC/Vsense_ADC
- J7 pad 1: /inverter/Vout_Inverter_- -> /inverter/Vout_Inverter_+
- J7 pad 2: /inverter/Vout_Inverter_+ -> /inverter/Vout_Inverter_-
- R22 pad 2: /ADC1_IN5 -> /currsense_DCDC/currsense_ADC
- R33 pad 1: VPP -> /voltsense_DCDC/Vsense_in
- R36 pad 2: /ADC1_IN0 -> /voltsense_DCDC/Vsense_ADC
- R4 pad 2: /ADC1_IN1 -> /voltsense_inverter/Vsense_ADC
- U1 pad 10: /TIM3_CH1 -> /inverter/Inv_Driver_Left_Hin
- U1 pad 12: /TIM3_CH2 -> /inverter/Inv_Driver_Left_Lin
- U2 pad 10: /TIM3_CH2 -> /inverter/Inv_Driver_Right_Hin
- U2 pad 12: /TIM3_CH1 -> /inverter/Inv_Driver_Right_Lin
- U3 pad 8: /ADC1_IN5 -> /currsense_DCDC/currsense_ADC

Commit message: im gonna start to route and probably revert to this version at least 5 times
Parts:
- added C17: C, Inductor_THT:L_Axial_L23.4mm_D12.7mm_P32.00mm_Horizontal_Vishay_IHA-203, F.Cu at (167.5, 154.7)
- added C20: C, Capacitor_THT:C_Rect_L24.0mm_W12.8mm_P22.50mm_MKT, F.Cu at (167.5, 127.4)
- added C3: C, Capacitor_THT:C_Rect_L32.0mm_W15.0mm_P27.00mm, F.Cu at (167.5, 125.2)
- added D23: LED, LED_SMD:LED_PLCC-2_3.4x3.0mm_AK, B.Cu at (55.0, 165.0)
- added D24: LED, LED_SMD:LED_PLCC-2_3.4x3.0mm_AK, B.Cu at (32.6, 166.0)
- added J12: Fuse holder or smth to hold tube, TestPoint:TestPoint_Loop_D2.60mm_Drill0.9mm_Beaded, B.Cu at (37.1, 151.6)
- added J13: Fuse holder or smth to hold tube, TestPoint:TestPoint_Loop_D2.60mm_Drill0.9mm_Beaded, B.Cu at (37.1, 156.7)
- added J14: Fuse holder or smth to hold tube, TestPoint:TestPoint_Loop_D2.60mm_Drill0.9mm_Beaded, B.Cu at (32.1, 151.6)
- added J15: Fuse holder or smth to hold tube, TestPoint:TestPoint_Loop_D2.60mm_Drill0.9mm_Beaded, B.Cu at (32.1, 156.7)
- added J27: Fuse holder or smth to hold tube, TestPoint:TestPoint_Loop_D2.60mm_Drill0.9mm_Beaded, F.Cu at (42.2, 151.6)
- added J28: Fuse holder or smth to hold tube, TestPoint:TestPoint_Loop_D2.60mm_Drill0.9mm_Beaded, B.Cu at (74.0, 177.6)
- added J29: Fuse holder or smth to hold tube, TestPoint:TestPoint_Loop_D2.60mm_Drill0.9mm_Beaded, B.Cu at (65.8, 170.2)
- added J30: Fuse holder or smth to hold tube, TestPoint:TestPoint_Loop_D2.60mm_Drill0.9mm_Beaded, B.Cu at (65.8, 175.3)
- added J31: Fuse holder or smth to hold tube, TestPoint:TestPoint_Loop_D2.60mm_Drill0.9mm_Beaded, B.Cu at (60.8, 170.2)
- added J32: Fuse holder or smth to hold tube, TestPoint:TestPoint_Loop_D2.60mm_Drill0.9mm_Beaded, B.Cu at (60.8, 175.3)
- added J33: Fuse holder or smth to hold tube, TestPoint:TestPoint_Loop_D2.60mm_Drill0.9mm_Beaded, B.Cu at (55.3, 170.6)
- added J34: Fuse holder or smth to hold tube, TestPoint:TestPoint_Loop_D2.60mm_Drill0.9mm_Beaded, B.Cu at (55.8, 175.3)
- added R58: R, Resistor_SMD:R_0805_2012Metric_Pad1.20x1.40mm_HandSolder, B.Cu at (31.2, 160.7)
- added R59: R, Resistor_SMD:R_0805_2012Metric_Pad1.20x1.40mm_HandSolder, B.Cu at (38.0, 163.6)
- C13, C14, C8, D11, D19, D20, D21, D22, D3, D6, HS1, HS2, HS3, HS4, HS5, HS6, J7, Q1, Q2, Q3, Q4, Q5, Q6, R12, R13, R15, R29, R30, R31, R32, R9: moved to B.Cu
- D9, R1, R2, R25, R26, R27, R44, R45, R8: moved to F.Cu
- moved R32 156.4 mm to (92.5, 160.6)
- moved R31 146.8 mm to (81.4, 151.8)
- moved D19 135.9 mm to (60.0, 140.0), turned to 180 degrees
- moved D20 135.4 mm to (52.6, 153.0), turned to 180 degrees
- moved R30 128.9 mm to (42.0, 143.7), turned to 180 degrees
- moved R29 128.9 mm to (42.0, 139.6), turned to 180 degrees
- moved D21 122.8 mm to (59.8, 145.9), turned to 180 degrees
- moved D22 117.5 mm to (50.0, 157.8), turned to 180 degrees
- moved C4 20.8 mm to (173.0, 138.6), turned to 0 degrees
- moved D4 13.3 mm to (202.6, 147.1), turned to 90 degrees
- moved D1 12.9 mm to (202.7, 135.3), turned to 90 degrees
- moved C15 12.5 mm to (194.0, 98.0), turned to 90 degrees
- moved C7 12.0 mm to (186.7, 142.7), turned to -90 degrees
- moved D9 9.66 mm to (198.8, 93.0), turned to -90 degrees
- moved D3 8.16 mm to (210.4, 129.5), turned to -90 degrees
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Connections:
- J7 pad 1: /inverter/Vout_Inverter_+ -> /inverter/Vout_Inverter_-
- J7 pad 2: /inverter/Vout_Inverter_- -> /inverter/Vout_Inverter_+
