File: WET_PCB_v2/voltsense_DCDC.kicad_sch (KiCad schematic)
At the start: 10 parts, among them J18 Capacitor connector, J20 Capacitor connector, U3 Opamp_Quad

Commit message: microcontroller to chip traces done
Parts:
- added R9: R0, Resistor_SMD:R_0805_2012Metric_Pad1.20x1.40mm_HandSolder, symbol Device:R
- D15: renamed from D30; footprint Diode_THT:D_DO-15_P2.54mm_Vertical_CathodeUp -> Diode_SMD:D_SMF
- D16: renamed from D29; footprint Diode_THT:D_DO-15_P2.54mm_Vertical_CathodeUp -> Diode_SMD:D_SMF
- J16: renamed from J18; footprint Connector_PinSocket_2.54mm:PinSocket_1x02_P2.54mm_Vertical -> Connector_PinSocket_2.54mm:PinSocket_1x02_P2.54mm_Horizontal
- renumbered J20 to J15, R33 to R39, R34 to R40, R35 to R41, R36 to R43, U3 to U1
Connections:
- net Vsense_ADC: now also R9.2; no longer J16.2 (Pin_2), R43.2
- new net: J16.2 (Pin_2), R43.2, R9.1
Other:
- moved on the sheet: J16
Changed lines of the file:
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@@
+	)
+	(junction
+		(at 111.76 63.5)
+		(diameter 0)
+		(color 0 0 0 0)
 	)
 	(junction
@@
 	)
 	(junction
-		(at 111.76 63.5)
-		(diameter 0)
-		(color 0 0 0 0)
-	)
-	(junction
 		(at 46.99 60.96)
 		(diameter 0)
@@
 	(wire
 		(pts
+			(xy 111.76 63.5) (xy 113.03 63.5)
+		)
+		(stroke
+			(width 0)
+			(type default)
+		)
+	)
+	(wire
+		(pts
 			(xy 55.88 73.66) (xy 55.88 76.2)
 		)
@@
 	(wire
 		(pts
+			(xy 120.65 63.5) (xy 121.92 63.5)
+		)
+		(stroke
+			(width 0)
+			(type default)
+		)
+	)
+	(wire
+		(pts
 			(xy 46.99 60.96) (xy 46.99 64.77)
 		)
@@
 	(wire
 		(pts
-			(xy 121.92 63.5) (xy 127 63.5)
+			(xy 121.92 63.5) (xy 142.24 63.5)
 		)
 		(stroke
@@
 		(pts
 			(xy 121.92 76.2) (xy 121.92 72.39)
-		)
-		(stroke
-			(width 0)
-			(type default)
-		)
-	)
-	(wire
-		(pts
-			(xy 111.76 63.5) (xy 121.92 63.5)
 		)
 		(stroke
@@
 	(hierarchical_label "Vsense_ADC"
 		(shape output)
-		(at 127 63.5 0)
+		(at 142.24 63.5 0)
 		(effects
 			(font
@@
 		(dnp no)
 		(fields_autoplaced yes)
-		(property "Reference" "D30"
+		(property "Reference" "D15"
 			(at 124.46 57.1499 90)
 			(show_name no)
@@
 			)
 		)
-		(property "Footprint" "Diode_THT:D_DO-15_P2.54mm_Vertical_CathodeUp"
+		(property "Footprint" "Diode_SMD:D_SMF"
 			(at 121.92 58.42 0)
 			(hide yes)
@@
 			(project "WET_PCB_v2"
 				(path "/13451c35-1666-47d9-9525-8d8125ba1cf3/a17383a4-d27f-4c25-9e0c-b0df1856b8d8"
-					(reference "D30")
+					(reference "D15")
 					(unit 1)
 				)
@@
 		(in_pos_files yes)
 		(dnp no)
-		(property "Reference" "#PWR056"
+		(property "Reference" "#PWR052"
 			(at 121.92 82.55 0)
 			(hide yes)
@@
 			(project "WET_PCB_v2"
 				(path "/13451c35-1666-47d9-9525-8d8125ba1cf3/a17383a4-d27f-4c25-9e0c-b0df1856b8d8"
-					(reference "#PWR056")
+					(reference "#PWR052")
 					(unit 1)
 				)
@@
 		(dnp no)
 		(fields_autoplaced yes)
-		(property "Reference" "R34"
+		(property "Reference" "R40"
 			(at 49.53 67.3099 0)
 			(show_name no)
@@
 			(project "WET_PCB_v2"
 				(path "/13451c35-1666-47d9-9525-8d8125ba1cf3/a17383a4-d27f-4c25-9e0c-b0df1856b8d8"
-					(reference "R34")
+					(reference "R40")
 					(unit 1)
 				)
@@
 		(dnp no)
 		(fields_autoplaced yes)
-		(property "Reference" "D29"
+		(property "Reference" "D16"
 			(at 124.46 67.3099 90)
 			(show_name no)
@@
 			)
 		)
-		(property "Footprint" "Diode_THT:D_DO-15_P2.54mm_Vertical_CathodeUp"
+		(property "Footprint" "Diode_SMD:D_SMF"
 			(at 121.92 68.58 0)
 			(hide yes)
@@
 			(project "WET_PCB_v2"
 				(path "/13451c35-1666-47d9-9525-8d8125ba1cf3/a17383a4-d27f-4c25-9e0c-b0df1856b8d8"
-					(reference "D29")
+					(reference "D16")
 					(unit 1)
 				)
@@
 		(dnp no)
 		(fields_autoplaced yes)
-		(property "Reference" "#PWR054"
+		(property "Reference" "#PWR050"
 			(at 55.88 82.55 0)
 			(hide yes)
@@
 			(project "WET_PCB_v2"
 				(path "/13451c35-1666-47d9-9525-8d8125ba1cf3/a17383a4-d27f-4c25-9e0c-b0df1856b8d8"
-					(reference "#PWR054")
+					(reference "#PWR050")
 					(unit 1)
 				)
@@
 		(dnp no)
 		(fields_autoplaced yes)
-		(property "Reference" "R35"
+		(property "Reference" "R41"
 			(at 63.5 54.61 90)
 			(show_name no)
@@
 			(project "WET_PCB_v2"
 				(path "/13451c35-1666-47d9-9525-8d8125ba1cf3/a17383a4-d27f-4c25-9e0c-b0df1856b8d8"
-					(reference "R35")
+					(reference "R41")
 					(unit 1)
 				)
@@
 		(in_pos_files yes)
 		(dnp no)
-		(property "Reference" "J20"
+		(property "Reference" "J15"
 			(at 58.42 66.0399 90)
 			(show_name no)
@@
 			(project "WET_PCB_v2"
 				(path "/13451c35-1666-47d9-9525-8d8125ba1cf3/a17383a4-d27f-4c25-9e0c-b0df1856b8d8"
-					(reference "J20")
+					(reference "J15")
 					(unit 1)
 				)
@@
 		(dnp no)
 		(fields_autoplaced yes)
-		(property "Reference" "R36"
+		(property "Reference" "R43"
 			(at 104.14 57.15 90)
 			(show_name no)
@@
 			(project "WET_PCB_v2"
 				(path "/13451c35-1666-47d9-9525-8d8125ba1cf3/a17383a4-d27f-4c25-9e0c-b0df1856b8d8"
-					(reference "R36")
+					(reference "R43")
 					(unit 1)
 				)
@@
 		(in_pos_files yes)
 		(dnp no)
-		(property "Reference" "U3"
+		(property "Reference" "U1"
 			(at 85.09 58.166 0)
 			(show_name no)
@@
 			(project "WET_PCB_v2"
 				(path "/13451c35-1666-47d9-9525-8d8125ba1cf3/a17383a4-d27f-4c25-9e0c-b0df1856b8d8"
-					(reference "U3")
+					(reference "U1")
 					(unit 1)
 				)
@@
 		(dnp no)
 		(fields_autoplaced yes)
-		(property "Reference" "R33"
+		(property "Reference" "R39"
 			(at 49.53 50.7999 0)
 			(show_name no)
@@
 			(project "WET_PCB_v2"
 				(path "/13451c35-1666-47d9-9525-8d8125ba1cf3/a17383a4-d27f-4c25-9e0c-b0df1856b8d8"
-					(reference "R33")
+					(reference "R39")
 					(unit 1)
 				)
@@
 		(in_pos_files yes)
 		(dnp no)
-		(property "Reference" "#PWR055"
+		(property "Reference" "#PWR051"
 			(at 111.76 82.55 0)
 			(hide yes)
@@
 			(project "WET_PCB_v2"
 				(path "/13451c35-1666-47d9-9525-8d8125ba1cf3/a17383a4-d27f-4c25-9e0c-b0df1856b8d8"
-					(reference "#PWR055")
+					(reference "#PWR051")
 					(unit 1)
 				)
@@
 	(symbol
 		(lib_id "Connector_Generic:Conn_02x01")
-		(at 111.76 71.12 90)
+		(at 111.76 71.12 270)
+		(mirror x)
 		(unit 1)
 		(body_style 1)
@@
 		(in_pos_files yes)
 		(dnp no)
-		(property "Reference" "J18"
-			(at 114.3 68.5799 90)
+		(property "Reference" "J16"
+			(at 109.22 68.5799 90)
 			(show_name no)
 			(do_not_autoplace no)
@@
 		)
 		(property "Value" "Capacitor connector"
-			(at 115.316 69.85 0)
+			(at 108.204 69.85 0)
 			(show_name no)
 			(do_not_autoplace no)
@@
 			)
 		)
-		(property "Footprint" "Connector_PinSocket_2.54mm:PinSocket_1x02_P2.54mm_Vertical"
+		(property "Footprint" "Connector_PinSocket_2.54mm:PinSocket_1x02_P2.54mm_Horizontal"
 			(at 111.76 71.12 0)
 			(hide yes)
@@
 			(project "WET_PCB_v2"
 				(path "/13451c35-1666-47d9-9525-8d8125ba1cf3/a17383a4-d27f-4c25-9e0c-b0df1856b8d8"
-					(reference "J18")
+					(reference "J16")
 					(unit 1)
 				)
@@
 		(dnp no)
 		(fields_autoplaced yes)
-		(property "Reference" "#PWR020"
+		(property "Reference" "#PWR049"
 			(at 46.99 82.55 0)
 			(hide yes)
@@
 			(project "WET_PCB_v2"
 				(path "/13451c35-1666-47d9-9525-8d8125ba1cf3/a17383a4-d27f-4c25-9e0c-b0df1856b8d8"
-					(reference "#PWR020")
+					(reference "#PWR049")
 					(unit 1)
 				)
@@
 					(unit 1)
 				)
+			)
+		)
+	)
+	(symbol
+		(lib_id "Device:R")
+		(at 116.84 63.5 90)
+		(unit 1)
+		(body_style 1)
+		(exclude_from_sim no)
+		(in_bom yes)
+		(on_board yes)
+		(in_pos_files yes)
+		(dnp no)
+		(fields_autoplaced yes)
+		(property "Reference" "R9"
+			(at 116.84 57.15 90)
+			(show_name no)
+			(do_not_autoplace no)
+			(effects
+				(font
+					(size 1.27 1.27)
+				)
+			)
+		)
+		(property "Value" "R0"
+			(at 116.84 59.69 90)
+			(show_name no)
+			(do_not_autoplace no)
+			(effects
+				(font
+					(size 1.27 1.27)
+				)
+			)
+		)
+		(property "Footprint" "Resistor_SMD:R_0805_2012Metric_Pad1.20x1.40mm_HandSolder"
+			(at 116.84 65.278 90)
+			(hide yes)
+			(show_name no)
+			(do_not_autoplace no)
+			(effects
+				(font
+					(size 1.27 1.27)
+				)
+			)
+		)
+		(property "Datasheet" ""
+			(at 116.84 63.5 0)
+			(hide yes)
+			(show_name no)
+			(do_not_autoplace no)
+			(effects
+				(font
+					(size 1.27 1.27)
+				)
+			)
+		)
+		(property "Description" "Resistor"
+			(at 116.84 63.5 0)
+			(hide yes)
+			(show_name no)
+			(do_not_autoplace no)
+			(effects
+				(font
+					(size 1.27 1.27)
+				)
+			)
+		)
+		(pin "2"
+		)
+		(pin "1"
+		)
+		(instances
+			(project "WET_PCB_v2"
+				(path "/13451c35-1666-47d9-9525-8d8125ba1cf3/a17383a4-d27f-4c25-9e0c-b0df1856b8d8"
+					(reference "R9")
+					(unit 1)
+				)

Commit message: labels
Parts:
- renumbered R42 to JMP20, R9 to JMP21
Changed lines of the file:
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@@
 		(dnp no)
 		(fields_autoplaced yes)
-		(property "Reference" "R42"
+		(property "Reference" "JMP20"
 			(at 83.82 64.77 90)
 			(show_name no)
@@
 			(project "WET_PCB_v2"
 				(path "/13451c35-1666-47d9-9525-8d8125ba1cf3/a17383a4-d27f-4c25-9e0c-b0df1856b8d8"
-					(reference "R42")
+					(reference "JMP20")
 					(unit 1)
 				)
@@
 		(dnp no)
 		(fields_autoplaced yes)
-		(property "Reference" "R9"
+		(property "Reference" "JMP21"
 			(at 116.84 57.15 90)
 			(show_name no)
@@
 			(project "WET_PCB_v2"
 				(path "/13451c35-1666-47d9-9525-8d8125ba1cf3/a17383a4-d27f-4c25-9e0c-b0df1856b8d8"
-					(reference "R9")
+					(reference "JMP21")
 					(unit 1)
 				)

Commit message: added values and notes for assembly
Parts:
- R39: value R -> 100kR
- R40: value R -> 5.1kR
- R41, R43: value R -> 0R
Changed lines of the file:
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@@
 			)
 		)
-		(property "Value" "R"
+		(property "Value" "5.1kR"
 			(at 49.53 69.8499 0)
 			(show_name no)
@@
 			)
 		)
-		(property "Value" "R"
+		(property "Value" "0R"
 			(at 63.5 57.15 90)
 			(show_name no)
@@
 			)
 		)
-		(property "Value" "R"
+		(property "Value" "0R"
 			(at 104.14 59.69 90)
 			(show_name no)
@@
 			)
 		)
-		(property "Value" "R"
+		(property "Value" "100kR"
 			(at 49.53 53.3399 0)
 			(show_name no)
@@
 		(in_pos_files yes)
 		(dnp no)
-		(fields_autoplaced yes)
 		(property "Reference" "JMP20"
-			(at 83.82 64.77 90)
+			(at 83.82 73.914 90)
 			(show_name no)
 			(do_not_autoplace no)
@@
 		)
 		(property "Value" "R0"
-			(at 83.82 67.31 90)
-			(show_name no)
-			(do_not_autoplace no)
+			(at 83.82 75.946 90)
+			(show_name no)
+			(do_not_autoplace no)
