File: WET_PCB_v2 - Copy/WET_PCB_v2.kicad_sch (KiCad schematic)
At the start: 38 parts, among them J1 Barrel jack, J10 POGO1, J11 Conn_01x09_Pin, J12 Conn_01x09_Pin, J2 Power input, J3 Jumper, J35 Programming, J36 LED_POWER, J4 Coil plug, J5 Vsense_ADC1_IN1, J6 Pluggable Terminal Block, J7 Conn_01x09_Pin, J8 Conn_01x09_Pin, J9 POGO2, U1 Opamp_Quad

Commit message: microcontroller to chip traces done
Parts:
- removed J35: Programming, Connector_PinSocket_2.54mm:PinSocket_1x02_P2.54mm_Horizontal, symbol Connector:Conn_01x02_Pin
- removed J36: LED_POWER, Connector_PinSocket_2.54mm:PinSocket_1x01_P2.54mm_Vertical, symbol Connector:Conn_01x01_Pin
- added D12: MBR1020VL, Diode_THT:D_DO-15_P2.54mm_Vertical_CathodeUp, symbol Diode:MBR1020VL
- added R54, R55, R56, R57: R0, Resistor_SMD:R_0805_2012Metric_Pad1.20x1.40mm_HandSolder, symbol Device:R
- J16: renamed from J10; footprint Connector_PinSocket_2.54mm:PinSocket_1x01_P2.54mm_Vertical -> Connector_PinHeader_1.00mm:PinHeader_1x01_P1.00mm_Vertical
- J21: renamed from J9; footprint Connector_PinSocket_2.54mm:PinSocket_1x01_P2.54mm_Vertical -> Connector_PinHeader_1.00mm:PinHeader_1x01_P1.00mm_Vertical
- renumbered C1 to C16, C2 to C18, C3 to C19, D1 to D13, D2 to D14, J8 to J10, J7 to J2, J5 to J26, J12 to J3, J2 to J4, J1 to J5, J4 to J6, J6 to J7, J3 to J8, R3 to R37, R8 to R38, R17 to R39, R20 to R40, R5 to R43, R14 to R44, R12 to R45, R6 to R48, R7 to R49, R1 to R5, R15 to R50, R16 to R51, R18 to R52, R19 to R53, R2 to R6, R4 to R7, R13 to R8, U1 to U3, U2 to U7
Connections:
- net ADC1_IN0: now also R55.2
- net ADC1_IN1: now also R57.2
- net ADC1_IN16: now also R56.2
- net ADC1_IN5: now also R54.2
- net DCDC/currsense_FET_side: now also R7.1; no longer R7.2
- net DCDC/currsense_cap_side: now also R7.2; no longer R7.1
- net VPP: now also D12.1 (K); no longer J4.1 (Pin_1)
- new net: D12.2 (A), J4.1 (Pin_1)
- new net curr_sense_coil/transducer_out_scaled: R56.1
- new net currsense_DCDC/currsense_ADC: R54.1
- new net voltsense_DCDC/Vsense_ADC: R55.1
- new net voltsense_inverter/Vsense_ADC: R57.1
Other:
- moved on the sheet: R38, R7
